File: kraftprom.kicad_sch (KiCad schematic)
At the start: 21 parts, among them J1 POWER, J2 PROGRAM, J3 Conn_01x04_Socket, U1 PIC16F628A, U2 74HC164, U3 74HC164, U4 74HC164, U5 74LS245, U6 74LS165

Commit message: KraftPROM
Parts:
- removed J1: POWER, symbol Connector:Conn_01x02_Socket
- removed J3: Conn_01x04_Socket, symbol Connector:Conn_01x04_Socket
- removed Z1: ZIF 28C16/28C64, Package_DIP:DIP-28_W15.24mm, symbol Memory_EEPROM:KM28C64A
- added U7: FTDI USB ADAPTER, symbol kraft80:FTDI-ADAPTER
- added Z1: ZIF 28 Pin, symbol kraft80:X28C64
- renumbered JP1 to J1
Connections:
- net +5V: now also U7.6 (5V), Z1.26 (NC), Z1.28 (VCC)
- net Earth: now also U7.16 (GND), U7.9 (GND), Z1.14 (GND)
- net ~{CE}: now also Z1.20 (~{CE})
- net ~{OE}: now also Z1.22 (~{OE})
- net ~{WE}: now also Z1.27 (~{WE})
- net at U2.10 (Q4): now also Z1.6 (A4)
- net at U2.11 (Q5): now also Z1.5 (A5)
- net at U2.12 (Q6): now also Z1.4 (A6)
- net at U2.13 (Q7), U3.1 (DSA), U3.2 (DSB): now also Z1.3 (A7)
- net at U2.3 (Q0): now also Z1.10 (A0)
- net at U2.4 (Q1): now also Z1.9 (A1)
- net at U2.5 (Q2): now also Z1.8 (A2)
- net at U2.6 (Q3): now also Z1.7 (A3)
- net at U5.11 (B7), U6.6 (D7): now also Z1.19 (I/O7)
- net at U5.12 (B6), U6.5 (D6): now also Z1.18 (I/O6)
- net at U5.13 (B5), U6.4 (D5): now also Z1.17 (I/O5)
- net at U5.14 (B4), U6.3 (D4): now also Z1.16 (I/O4)
- net at U5.15 (B3), U6.14 (D3): now also Z1.15 (I/O3)
- net at U5.16 (B2), U6.13 (D2): now also Z1.13 (I/O2)
- net at U5.17 (B1), U6.12 (D1): now also Z1.12 (I/O1)
- net at U5.18 (B0), U6.11 (D0): now also Z1.11 (I/O0)
- net at U1.2 (RA3/AN3/CMP1): now also U7.12 (~{RTS})
- net at U1.7 (RB1/RX/DT): now also U7.10 (TXD)
- net at U1.8 (RB2/TX/CK): now also U7.14 (RXD)
- net at U3.10 (Q4): now also Z1.2 (A12)
- net at U3.5 (Q2): now also Z1.21 (A10)
- net at J1.2 (C): now also Z1.23 (A11)
- net at U3.4 (Q1): now also Z1.24 (A9)
- net at U3.3 (Q0): now also Z1.25 (A8)
Other:
- note removed: "CTS"
- note removed: "Connect PIN26 to VCC"
- note removed: "GND"
- note removed: "If using a USB serial adapter, most likely it will already have a +5V output with a good decoupling capacitor. This is the recommended option."
- note removed: "RX"
- note removed: "TTL 5V levels for use with USB adapters or TTL/RS converters."
- note removed: "TX"
- moved on the sheet: C1, C2, C3, C7, C8, J2, U1

Commit message: More PCB design (fixes).
Connections:
- net at U7.12 (~{RTS}): no longer U1.2 (RA3/AN3/CMP1)
- net at U7.4 (~{CTS}): now also U1.2 (RA3/AN3/CMP1)
Changed lines of the file:
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@@
+	(wire
+		(pts
+			(xy 46.99 189.23) (xy 46.99 194.31)
+		)
+		(stroke
+			(width 0)
+			(type default)
+		)
+	)
 	(wire
 		(pts
@@
 	(wire
 		(pts
-			(xy 54.61 156.21) (xy 54.61 166.37)
-		)
-		(stroke
-			(width 0)
-			(type default)
-		)
-	)
-	(wire
-		(pts
 			(xy 124.46 43.18) (xy 125.73 43.18)
 		)
@@
 	(wire
 		(pts
+			(xy 46.99 194.31) (xy 16.51 194.31)
+		)
+		(stroke
+			(width 0)
+			(type default)
+		)
+	)
+	(wire
+		(pts
 			(xy 125.73 73.66) (xy 125.73 82.55)
 		)
@@
 	(wire
 		(pts
+			(xy 16.51 194.31) (xy 16.51 156.21)
+		)
+		(stroke
+			(width 0)
+			(type default)
+		)
+	)
+	(wire
+		(pts
 			(xy 21.59 57.15) (xy 29.21 57.15)
 		)
@@
 	(wire
 		(pts
-			(xy 49.53 156.21) (xy 54.61 156.21)
-		)
-		(stroke
-			(width 0)
-			(type default)
-		)
-	)
-	(wire
-		(pts
 			(xy 217.17 53.34) (xy 217.17 68.58)
 		)
@@
 		)
 		(stroke
+			(width 0)
+			(type default)
+		)
+	)
+	(wire
+		(pts
+			(xy 16.51 156.21) (xy 49.53 156.21)
+		)
+		(stroke
